File: pcb/BPV4_Collar/BPV4_Collar.kicad_sch (KiCad schematic)
At the start: 32 parts, among them IC1 RAK4630, IC2 GM02SP, J1 Conn_01x03, J2 Conn_01x05, J3 USB_C_Receptacle_USB2.0_14P, J4 Conn_01x08, J5 Conn_01x08, U1 BQ24074RGT, U2 TPS62840DLCR, U3 MAX17048G_T10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

Commit message: pcb design 80% complete
Parts:
- added C12: 100nF, symbol Device:C
- added D1: LED, symbol Device:LED
- added J6: SIM8055-6-1-14-00-A, SIM8055-6-1-14-00-A:GCT_SIM8055-6-1-14-00-A, symbol SIM8055-6-1-14-00-A:SIM8055-6-1-14-00-A
- added J7: CONUFL001-SMD-T, CONUFL001SMDT, symbol CONUFL001-SMD-T:CONUFL001-SMD-T
- added JP1: SJ_2_Open, symbol Jumper:SolderJumper_2_Open
- added L2: LQW03AW10NJ00D, LQW03AW10NJ00D, symbol LQW03AW10NJ00D:LQW03AW10NJ00D
- added R10, R11, R14, R15: 100k, symbol Device:R
- added R12: 1k, symbol Device:R
- added R13: 4.7k, symbol Device:R
- added R16: 0RO, symbol Device:R
- added R17, R18: DNP, symbol Device:R
- added T1: NX3008PBKMB, NX3008PBKMB:SOT883_B_, symbol NX3008PBKMB:NX3008PBKMB
- added TP1: RTS1, symbol Connector:TestPoint
- added TP2: RXD1, symbol Connector:TestPoint
- added TP3: CTS1, symbol Connector:TestPoint
- added TP4: TXD1, symbol Connector:TestPoint
- added TP5: RES_FFF/FFH, symbol Connector:TestPoint
- added TP6: RXD2, symbol Connector:TestPoint
- added TP8: TXD2, symbol Connector:TestPoint
Connections:
- net GM02SP_CTS is gone; now on net RESETN: J5.8 (Pin_8)
- net GM02SP_RTS is gone; now on net WAKE0: J5.7 (Pin_7)
- net GM02SP_UART_RX is gone; now on net UART0_RX: J5.4 (Pin_4)
- net GM02SP_UART_TX is gone; now on net UART0_TX: J5.5 (Pin_5)
- net RAK_RTS is gone; now on net WAKE: J4.7 (Pin_7)
- net RAK_UART_RX is gone; now on net UART_RX: J4.5 (Pin_5)
- net RAK_UART_TX is gone; now on net UART_TX: J4.4 (Pin_4)
- net Receive_PWRKEY_RSET is gone; now on net PS_STATUS: J5.6 (Pin_6)
- net SEND_PWRKEY_RSET is gone; now on net GM02SP_PS_STATUS: J4.6 (Pin_6)
- net BAT_NTC: no longer R1.2, U1.1 (TS)
- net Batt_I2C_SCL: no longer IC1.4 (P0.13/I2C_SDA)
- net Batt_I2C_SDA: no longer IC1.5 (P0.14/I2C_SCL)
- net GND: now also C12.2, D1.1 (K), J6.C4 (SHIELD), J6.C5 (GND), J6.C8 (SHIELD__1), J7.2 (GND_1), J7.3 (GND_2), R10.1, R11.1, R15.1, R17.1, R18.1
- net SWDCLK: now also IC1.19 (SWDIO); no longer IC1.18 (SWDCLK)
- net SWDIO: now also IC1.18 (SWDCLK); no longer IC1.19 (SWDIO)
- net WAKE: no longer J4.3 (Pin_3)
- net WAKE0: now also IC2.48 (WAKE0); no longer J5.3 (Pin_3)
- net at IC2.12 (GPIO1/_STATUS_LED): now also R12.1
- net PS_STATUS: now reaches IC2.13 (GPIO2/_PS_STATUS)
- net PS_STATUS: now also R10.2
- net GNSS_EN: now reaches IC2.14 (GPIO28/_DTR0)
- net at IC2.20 (RESERVED/_FFF_FFH): now also R11.2, TP5.1
- net at IC2.26 (GPIO16/RXD2): now also TP6.1
- net at IC2.28 (GPIO15/TXD2): now also TP8.1
- net at IC2.29 (RTS1): now also TP1.1
- net at IC2.30 (RXD1): now also TP2.1
- net at IC2.31 (CTS1): now also TP3.1
- net at IC2.32 (TXD1): now also TP4.1
- net UART0_RX: now reaches IC2.34 (GPIO13/RXD0)
- net UART0_TX: now reaches IC2.36 (GPIO12/TXD0)
- net SIM_CLK: now reaches IC2.42 (SIM0_CLK)
- net SIM_CLK: now also J6.C3 (CLK)
- net SIM_RSET: now reaches IC2.43 (SIM0_RSTN)
- net SIM_RSET: now also J6.C2 (RST)
- net SIM_IO: now reaches IC2.44 (SIM0_IO)
- net SIM_IO: now also IC2.73 (SIM0_VCC), C12.1, J6.C1 (VCC), R13.2
- net RESETN: now reaches IC2.46 (RESETN)
- net 1V8_OUT: now reaches IC2.8 (1V8)
- net 1V8_OUT: now also R14.2, T1.3
- net GM02SP_PS_STATUS: now reaches IC1.39 (P0.31/AIN7)
- net Batt_Alert renamed USB_D+
- net USB_D+: no longer U3.5 (~{ALERT})
- net RAK_CTS renamed GM02SP_RESET
- new net: D1.2 (A), JP1.1 (A)
- new net: JP1.2 (B), R12.2
- new net: J6.CD, R14.1, T1.1
- new net: J6.C7 (I/O), R13.1
- new net: L2.2, R16.2, R18.2
- new net: J7.1 (SIG), R16.1, R17.2
- new net BATT_ALERT: U3.5 (~{ALERT})
- new net BATT_I2C_SCL: IC1.5 (P0.14/I2C_SCL)
- new net BATT_I2C_SDA: IC1.4 (P0.13/I2C_SDA)
- new net BATT_NTC: R1.2, U1.1 (TS)
- new net SIM_DETECT: R15.2, T1.2
- no-connect marks 9 -> 47
Other:
- note added: "'Fuel guage' Battery level monitor"
- note added: "(5V sense only; not for 5V power supply)"
- note added: "(sim card holder/ socket)"
- note added: "JST 3pin Battery terminal"
- note added: "LiPo Battery charger IC"
- note added: "Monarch 2 GM02SP"
- note added: "RAK4630 (NRF52840 MCU + SX1262 LoRa)"
- note added: "VBAT Regulator (LiPo 3.0V~4.2V to stable VCC_3.3v for system)"
- note added: "single wire debug (SWD)socket"
- moved on the sheet: C10, C4, C5, C6, C9, R1, R7
