File: pcb/BPV4_Collar/BPV4_Collar.kicad_sch (KiCad schematic)
At the start: 55 parts, among them IC1 RAK4630, IC2 GM02SP, J1 Conn_01x03, J2 Conn_01x05, J3 USB_C_Receptacle_USB2.0_14P, J4 Conn_01x08, J5 Conn_01x08, J6 SIM8055-6-1-14-00-A, J7 CONUFL001-SMD-T, T1 NX3008PBKMB, U1 BQ24074RGT, U2 TPS62840DLCR, U3 MAX17048G_T10, U4 USBLC6-2SC6

Commit message: Update KiCad PCB designs and component libraries
Parts:
- removed C10: C 100nF, symbol Device:C
- removed C8: 10nF, symbol Device:C
- removed IC2: GM02SP, GM02SP, symbol GM02SP_lib:GM02SP
- removed J5: Conn_01x08, symbol Connector_Generic:Conn_01x08
- removed J6: SIM8055-6-1-14-00-A, SIM8055-6-1-14-00-A:GCT_SIM8055-6-1-14-00-A, symbol SIM8055-6-1-14-00-A:SIM8055-6-1-14-00-A
- removed J7: CONUFL001-SMD-T, CONUFL001SMDT, symbol CONUFL001-SMD-T:CONUFL001-SMD-T
- removed JP1: SJ_2_Open, symbol Jumper:SolderJumper_2_Open
- removed L2: LQW03AW10NJ00D, LQW03AW10NJ00D, symbol LQW03AW10NJ00D:LQW03AW10NJ00D
- removed R1: 10k, symbol Device:R
- removed R11: 100k, symbol Device:R
- removed R12: 1k, symbol Device:R
- removed R18: DNP, symbol Device:R
- removed T1: NX3008PBKMB, NX3008PBKMB:SOT883_B_, symbol NX3008PBKMB:NX3008PBKMB
- removed TP1: RTS1, symbol Connector:TestPoint
- removed TP2: RXD1, symbol Connector:TestPoint
- removed TP3: CTS1, symbol Connector:TestPoint
- removed TP4: TXD1, symbol Connector:TestPoint
- removed TP5: RES_FFF/FFH, symbol Connector:TestPoint
- removed TP6: RXD2, symbol Connector:TestPoint
- removed TP8: TXD2, symbol Connector:TestPoint
- added BZ1: CPT-7502-65-SMT-TR, CPT-7502-65-SMT-TR:XDCR_CPT-7502-65-SMT-TR, symbol CPT-7502-65-SMT-TR:CPT-7502-65-SMT-TR
- added C13, C3: 100nF, Capacitor_SMD:C_0402_1005Metric, symbol Device:C
- added C14: 10uF, Capacitor_SMD:C_0201_0603Metric, symbol Device:C
- added D2: DMG2305UX-13, LIB_DMG2305UX-13:SOT96P240X120-3N, symbol DMG2305UX-13:DMG2305UX-13
- added D3, D4: LED, LED_SMD:LED_0402_1005Metric, symbol Device:LED
- added FID1, FID2, FID3: Fiducial, Fiducial:Fiducial_0.5mm_Mask1mm, symbol Mechanical:Fiducial
- added J3: Conn_01x04, Connector_PinHeader_2.54mm:PinHeader_1x04_P2.54mm_Vertical, symbol Connector_Generic:Conn_01x04
- added J6: Conn_01x06, Connector:Tag-Connect_TC2030-IDC-NL_2x03_P1.27mm_Vertical, symbol Connector_Generic:Conn_01x06
- added J7: Conn_01x02_Pin, Connector_PinHeader_1.00mm:PinHeader_1x02_P1.00mm_Vertical, symbol Connector:Conn_01x02_Pin
- added MH1, MH2: M2_Screw, MountingHole:MountingHole_2.2mm_M2_Pad_Via, symbol Mechanical:MountingHole_Pad
- added R6: 1M, Resistor_SMD:R_0402_1005Metric, symbol Device:R
- added R8, R9: 10k, Resistor_SMD:R_0402_1005Metric, symbol Device:R
- added SW1, SW2: SW_Push, Button_Switch_SMD:SW_SPST_B3U-1000P, symbol B3U-1000P:B3U-1000P
- added U6: LIS2DW12TR, LIS2DW12TR:LGA12R50P4X4_200X200X70, symbol LIS2DW12TR:LIS2DW12TR
- C1: footprint (none) -> Capacitor_SMD:C_0201_0603Metric
- C10: renamed from C6; value C 100nF -> 100nF; footprint (none) -> Capacitor_SMD:C_0402_1005Metric
- C11: renamed from C7; value C 10uF -> 10uF; footprint (none) -> Capacitor_SMD:C_0201_0603Metric
- C12: footprint (none) -> Capacitor_SMD:C_0402_1005Metric
- C2: renamed from C11; footprint (none) -> Capacitor_SMD:C_0402_1005Metric
- C4: renamed from C3; value C 10uF -> 10uF; footprint (none) -> Capacitor_SMD:C_0201_0603Metric
- C5: renamed from C2; value C 10uF -> 10uF; footprint (none) -> Capacitor_SMD:C_0201_0603Metric
- C6: renamed from C9; footprint (none) -> Capacitor_SMD:C_0402_1005Metric
- C8: renamed from C4; value C 100nF -> 1uF; footprint (none) -> Capacitor_SMD:C_0402_1005Metric
- C9: renamed from C5; value C 100nF -> 100nF; footprint (none) -> Capacitor_SMD:C_0402_1005Metric
- D1: footprint (none) -> LED_SMD:LED_0402_1005Metric
- IC1: footprint RAK4630 -> RAK4630:RAK4630
- J1: footprint (none) -> Connector_JST:JST_SH_SM03B-SRSS-TB_1x03-1MP_P1.00mm_Horizontal
- J2: footprint (none) -> Connector_PinHeader_1.00mm:PinHeader_1x05_P1.00mm_Vertical
- J4: renamed from J3; footprint (none) -> Connector_USB:USB_C_Receptacle_GCT_USB4105-xx-A_16P_TopMnt_Horizontal; symbol Connector:USB_C_Receptacle_USB2.0_14P -> Connector:USB_C_Receptacle_USB2.0_16P
- J5: renamed from J4; footprint (none) -> Connector_JST:JST_SH_SM08B-SRSS-TB_1x08-1MP_P1.00mm_Horizontal
- L1: footprint (none) -> Inductor_SMD:L_0201_0603Metric
- R1: renamed from R5; footprint (none) -> Resistor_SMD:R_0402_1005Metric
- R10, R14: value 100k -> 1k; footprint (none) -> Resistor_SMD:R_0402_1005Metric
- R11: renamed from R8; footprint (none) -> Resistor_SMD:R_0402_1005Metric
- R12: renamed from R9; footprint (none) -> Resistor_SMD:R_0402_1005Metric
- R13: value 4.7k -> 1k; footprint (none) -> Resistor_SMD:R_0402_1005Metric
- R15: value 100k -> 10k; footprint (none) -> Resistor_SMD:R_0402_1005Metric
- R16: value 0RO -> 10k; footprint (none) -> Resistor_SMD:R_0402_1005Metric
- R17: value DNP -> 1k; footprint (none) -> Resistor_SMD:R_0402_1005Metric
- R2: footprint (none) -> Resistor_SMD:R_0402_1005Metric
- R3: renamed from R4; footprint (none) -> Resistor_SMD:R_0402_1005Metric
- R4: renamed from R6; footprint (none) -> Resistor_SMD:R_0402_1005Metric
- R5: renamed from R3; footprint (none) -> Resistor_SMD:R_0402_1005Metric
- R7: value 10k -> 1M; footprint (none) -> Resistor_SMD:R_0402_1005Metric
- renumbered U3 to U1, U1 to U2, U2 to U3
Connections:
- net BAT_NTC is gone; now on net BATT_NTC: J1.3 (Pin_3)
- net Batt_I2C_SCL is gone; now on net BATT_I2C_SCL: R3.1, U1.7 (SCL)
- net Batt_I2C_SDA is gone; now on net BATT_I2C_SDA: R1.2, U1.8 (SDA)
- net SIM_DETECT is gone; now on an unnamed net: R15.2
- net BATT_ALERT: now also IC1.11 (P0.21/UART1_DE)
- net GM02SP_PS_STATUS: now also IC1.10 (P0.20/UART1_TX_(AT_COMMAND)); no longer IC1.39 (P0.31/AIN7)
- net GM02SP_RESET: now also IC1.9 (P0.19/UART1_RX_(AT_COMMAND))
- net GND: now also J5.3 (Pin_3), R7.1, R7.2, BZ1.1, C13.2, C14.2, C3.2, D2.1 (G), D3.1 (K), D4.1 (K), J3.1 (Pin_1), J6.5 (Pin_5), J6.6 (Pin_6), SW1.2 (A), SW2.1 (K), U6.2 (CS), U6.3 (SDO/SA0), U6.6 (GND), U6.7 (RES), U6.8 (GND); no longer C1.1, IC1.35 (GND_4), J1.1 (Pin_1), J2.2 (Pin_2), J5.1 (Pin_1), R10.1, R15.1, R17.1, U1.2 (CELL), U2.2 (BAT), U2.3 (BAT), U3.2 (VIN), U3.4 (EN)
- net NRF_RESET: now also J6.3 (Pin_3); no longer J2.5 (Pin_5), R7.1
- net SWDCLK: now also IC1.18 (SWDCLK), J6.4 (Pin_4); no longer IC1.19 (SWDIO), J2.4 (Pin_4)
- net SWDIO: now also IC1.19 (SWDIO), J6.2 (Pin_2); no longer IC1.18 (SWDCLK), J2.3 (Pin_3)
- net UART_RX: now also J3.4 (Pin_4)
- net UART_TX: now also J3.3 (Pin_3)
- net VCC_3v3: now also IC1.21 (VBAT_IO_SX), R15.1, R16.1, C13.1, C14.1, J3.2 (Pin_2), J6.1 (Pin_1), R8.1, R9.1, U6.10 (VDDIO), U6.9 (VDD); no longer C11.1, IC1.43 (VDD_NRF), IC1.44 (VBAT_NRF), J2.1 (Pin_1), R7.2
- net WAKE: now also IC1.8 (P0.17/UART2_DE)
- net at D1.2 (A): now also R13.2
- net at R14.1: now also IC1.30 (P0.02/QSPI_DIO3)
- net at R13.1: now also IC1.27 (P1.03/LED1)
- net at R16.2: now also IC1.23 (P0.24/I2C_SDA_2), U6.4 (SDA/SDI/SDO)
- net at R17.2: now also D3.2 (A); no longer R16.1
- net at IC1.12 (P0.10/NFC2): now also J7.1 (Pin_1)
- net at IC1.13 (P0.09/NFC1): now also J7.2 (Pin_2)
- net at IC1.24 (P0.25/I2C_SCL_2): now also U6.1 (SCL/SPC)
- net at IC1.25 (P1.01/SW1): now also R9.2, SW2.2 (A)
- net at IC1.26 (P1.02/SW2): now also R8.2, SW1.1 (K)
- net at IC1.28 (P1.04/LED2): now also R17.1
- net at IC1.29 (P0.03/QSPI_CLK): now also R10.1
- net at IC1.31 (P0.28/QSPI_DIO2): now also J2.5 (Pin_5)
- net at IC1.32 (P0.29/QSPI_DIO1): now also J2.4 (Pin_4)
- net at IC1.33 (P0.30/QSPI_DIO0): now also J2.3 (Pin_3)
- net at IC1.34 (P0.26/QSPI_CS): now also J2.2 (Pin_2)
- net Accel: now reaches IC1.40 (P0.05/AIN3)
- net Accel: now also U6.12 (INT1)
- net VBAT_SENSE: now reaches IC1.41 (P0.04/AIN2)
- net VBAT_SENSE: now also C3.1, R6.1
- net VOUT_SYS: now reaches U2.10 (OUT), U2.11 (OUT)
- net VOUT_SYS: now also C1.1, C11.1, C12.1, IC1.44 (VBAT_NRF), J5.1 (Pin_1), U3.2 (VIN), U3.4 (EN)
- net 1V8_OUT: no longer names the net of R14.2
- net 1V8_OUT: now also BZ1.2
- net PS_STATUS: no longer names the net of R10.2
- net PS_STATUS: now also D4.2 (A)
- removed net SIM_IO: C12.1, R13.2
- new net: IC1.35 (GND_4), J2.1 (Pin_1)
- new net VBAT: D2.3 (D), R6.2, U1.2 (CELL), U2.2 (BAT), U2.3 (BAT)
- new net VBAT_RAW+: D2.2 (S), J1.1 (Pin_1)
- no-connect marks 47 -> 14
Other:
- note added: "(5V sense only. Not for 5V power supply)"
- note added: "3v3 Buck Regulator Input: VOUT_SYS from BQ24074 OUT Converts to stable/constant VCC_3.3v for the system"
- note added: "JST SH 1.0mm pitch 8-Pin Ribbon wire connection"
- note added: "MEMS Accelerometer"
- note added: "NFC1 pad?"
- note added: "NFC2 pad?"
- note added: "Need to verify this is correct & conventional way to do ESD/Diode <-----"
- note added: "Page 1of2 RAK4630(NRF52840 MCU +SX1262 Lora RFIC)"
- note added: "RAK4630 (NRF52840 MCU + SX1262 LoRa) (Using presoldered Ipex connectors for BT/LoRa)"
- note added: "UART_2 to GM02sp"
- note added: "Voltage divider 2:1 For RAK4630 AIN2/P0.04 Backup Voltage measurement"
- note added: "takes 5v from USB, outputs to: Pin:2VBAT>DMG230_Diode>Pin2:VBAT_RAW(to charge the battery) Pin10:VOUT_SYS > TPS6284_BUCK Pin2: VIN"
- note removed: "(5V sense only; not for 5V power supply)"
- note removed: "(sim card holder/ socket)"
- note removed: "Monarch 2 GM02SP"
- note removed: "Monarch 2 GM02SP Module (CAT-M/NB-IoT + GNSS Receiver)"
- note removed: "RAK4630 (NRF52840 MCU + SX1262 LoRa)"
- note removed: "RAK4630(NRF52840 MCU +SX1262 Lora RFIC)"
- note removed: "Tx>Rx= =Rx>Tx"
- note removed: "VBAT Regulator (LiPo 3.0V~4.2V to stable VCC_3.3v for system)"
- moved on the sheet: C1, C10, C11, C2, C4, C5, C6, C8, C9, IC1, J1, L1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
