File: pcb/collar/BPV4_Collar/All_In_One_collar_sch.kicad_sch (KiCad schematic)
At the start: 86 parts, among them IC1 RAK4630, IC3 SKY65723-11, IC5 GM02SP, J1 Conn_01x03, J10 CONUFL001-SMD-T, J13 SIM8055-6-1-14-00-A, J2 Conn_01x05, J3 Conn_01x04, J4 USB_C_Receptacle_USB2.0_14P, J5 Conn_01x04, J6 Conn_01x06, J7 Conn_01x02_Pin, J9 CONUFL001-SMD-T, SW1 SW_Push, SW2 SW_Push, T2 NX3008PBKMB, U1 MAX17048G_T10, U2 BQ24074RGT, U3 TPS62840DLCR, U4 USBLC6-2SC6, U6 LIS2DW12TR

Commit message: Update integrated collar PCB design
Parts:
- removed R19: 267K, Resistor_SMD:R_0402_1005Metric, symbol Device:R
Connections:
- net GND: now also U3.5 (VSET), U6.2 (CS); no longer U2.4 (~{CE})
- net VCC_3v3: now also U2.4 (~{CE})
- net at IC1.23 (P0.24/I2C_SDA_2), R15.2, U6.1 (SCL/SPC): no longer U6.2 (CS)
Other:
- moved on the sheet: C16, C17, C20, C21, D5, FID1, FID2, FID3, IC5, J13, J5, J9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
