File: pcb/collar/BPV4_Collar/BPV4_Collar.kicad_sch (KiCad schematic)
At the start: 86 parts, among them IC1 RAK4630, IC3 SKY65723-11, IC5 GM02SP, J1 Conn_01x03, J10 CONUFL001-SMD-T, J13 SIM8055-6-1-14-00-A, J2 Conn_01x05, J3 Conn_01x04, J4 USB_C_Receptacle_USB2.0_14P, J5 Conn_01x04, J6 Conn_01x06, J7 Conn_01x02_Pin, J9 CONUFL001-SMD-T, SW1 SW_Push, SW2 SW_Push, T2 NX3008PBKMB, U1 MAX17048G_T10, U2 BQ24074RGT, U3 TPS62840DLCR, U4 USBLC6-2SC6, U6 LIS2DW12TR

Commit message: Save ST4SIM-300M schematic work in progress
Parts:
- removed FID4, FID5, FID6: Fiducial, Fiducial:Fiducial_0.5mm_Mask1mm, symbol Mechanical:Fiducial
- removed H1, H2: MountingHole_Pad, MountingHole:MountingHole_2.2mm_M2_Pad_Via, symbol Mechanical:MountingHole_Pad
- removed J13: SIM8055-6-1-14-00-A, SIM8055-6-1-14-01-A:SIM8055611401A, symbol SIM8055-6-1-14-00-A:SIM8055-6-1-14-00-A
- removed J3: Conn_01x04, Connector_PinHeader_2.54mm:PinHeader_1x04_P2.54mm_Vertical, symbol Connector_Generic:Conn_01x04
- removed J5: Conn_01x04, Connector_PinSocket_2.54mm:PinSocket_1x04_P2.54mm_Vertical, symbol Connector_Generic:Conn_01x04
- removed R38, R41: 100k, Resistor_SMD:R_0603_1608Metric, symbol Device:R
- removed R4: 10k, Resistor_SMD:R_0402_1005Metric, symbol Device:R
- removed R42: 4.7k, Resistor_SMD:R_0603_1608Metric, symbol Device:R
- removed T2: NX3008PBKMB, NX3008NBKW_115:SOT65P210X110-3N, symbol NX3008PBKMB:NX3008PBKMB
- added C18: 1uF, Capacitor_SMD:C_0201_0603Metric, symbol Device:C
- added IC2: ST4SI3M004600HFW, SON127P600X500X100-9N, symbol ST4SI3M004600HFW:ST4SI3M004600HFW
- added R20: 4.7k, Resistor_SMD:R_0402_1005Metric, symbol Device:R
- added R32: 20k, Resistor_SMD:R_0603_1608Metric, symbol Device:R
- added R34: 100k, Resistor_SMD:R_0603_1608Metric, symbol Device:R
- C6: value C 100nF -> 100nF
- R2: value 1k -> 3.48k
- R5: value 1k -> 2.2k
- renumbered D2 to Q2
Connections:
- net PS_STATUS is gone; now on net GM02SP_PS_STATUS: IC5.13 (GPIO2/_PS_STATUS), R35.2
- net RESETN is gone; now on net GM02SP_RESET: IC5.46 (RESETN)
- net UART0_RX is gone; now on net UART_TX: IC5.34 (GPIO13/RXD0)
- net UART0_TX is gone; now on net UART_RX: IC5.36 (GPIO12/TXD0)
- net WAKE0 is gone; now on net WAKE: IC5.48 (WAKE0)
- net BATT_ALERT: now also R20.2
- net GND: now also U1.1 (CTG), U1.6 (QSTRT), C18.2, IC2.1 (GND); no longer R7.2, U2.14 (TMR), U2.6 (EN1)
- net SIM_CLK: now also IC2.6 (CLK)
- net SIM_IO: now also IC2.3 (I/O), R32.1
- net SIM_RESET: now also IC2.7 (~{RESET})
- net VBAT: now also C6.1, Q2.2 (S), U1.3 (VDD); no longer C16.1, C17.1, C20.1, IC5.60 (VBAT_1), IC5.62 (VBAT_2), IC5.63 (VBAT_3), Q2.3 (D)
- net VBAT_RAW+: now also Q2.3 (D); no longer Q2.2 (S)
- net VBAT_SENSE: now also R7.2
- net VCC_3v3: now also U2.6 (EN1), R20.1; no longer C6.1, U1.3 (VDD)
- net VOUT_SYS: now also C16.1, C17.1, C20.1, IC5.60 (VBAT_1), IC5.62 (VBAT_2), IC5.63 (VBAT_3), R34.2
- net VSIM: now also C18.1, IC2.8 (VCC), R32.2
- net SIM_DETECT: no longer names the net of IC5.45 (SIM0_DETECT)
- net SIM_DETECT: now also R34.1
- no-connect marks 67 -> 69
Other:
- note added: "<--Verify EP connection before PCB release"
- note removed: "(NanoSim card holder socket)"
- note removed: "UART_2 to GM02sp"
- moved on the sheet: C13, C14, C3, C6, Q2, R15, R16, R24, R26, R28, R31, R7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
